File: SRAD_computer/_autosave-SRAD_computer.kicad_sch (KiCad schematic)
At the start: 49 parts, among them J1 USB_B_Micro, J2 Conn_01x02, U1 NCP1117-3.3_SOT223, U2 W25Q128JVS, U3 RP2040, U4 BME280, U5 MPU-9250, U6 SAM-M8Q-0-10, Y1 ABM8-272-T3

Commit message: PCB placement
Parts:
- C_BME_VDDIO1, C_MPU_REG1: footprint TCLib:C_5mm -> TCLib:C_0805
- C_MPU_VDD: renamed from C_VDD_MPU1; footprint TCLib:C_5mm -> TCLib:C_0805
- C_MPU_VDDIO: renamed from C_VDDIO_MPU1; footprint TCLib:C_5mm -> TCLib:C_0805
Changed lines of the file:
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@@
 			)
 		)
-		(property "Footprint" "TCLib:C_5mm"
+		(property "Footprint" "TCLib:C_0805"
 			(at 81.28 248.158 0)
 			(effects
@@
 			)
 		)
-		(property "Description" "Unpolarized capacitor"
+		(property "Description" ""
 			(at 80.518 243.586 0)
 			(effects
@@
 		(dnp no)
 		(fields_autoplaced yes)
-		(property "Reference" "C_VDDIO_MPU1"
+		(property "Reference" "C_MPU_VDDIO"
 			(at 114.3 240.0299 0)
 			(effects
@@
 			)
 		)
-		(property "Footprint" "TCLib:C_5mm"
+		(property "Footprint" "TCLib:C_0805"
 			(at 93.98 237.998 0)
 			(effects
@@
 			)
 		)
-		(property "Description" "Unpolarized capacitor"
+		(property "Description" ""
 			(at 93.218 233.426 0)
 			(effects
@@
 			(project ""
 				(path "/f015d259-36b1-4d36-b25a-c9dc3131b66c"
-					(reference "C_VDDIO_MPU1")
+					(reference "C_MPU_VDDIO")
 					(unit 1)
 				)
@@
 		(dnp no)
 		(fields_autoplaced yes)
-		(property "Reference" "C_VDD_MPU1"
+		(property "Reference" "C_MPU_VDD"
 			(at 97.79 226.0599 0)
 			(effects
@@
 			)
 		)
-		(property "Footprint" "TCLib:C_5mm"
+		(property "Footprint" "TCLib:C_0805"
 			(at 77.47 224.028 0)
 			(effects
@@
 			)
 		)
-		(property "Description" "Unpolarized capacitor"
+		(property "Description" ""
 			(at 76.708 219.456 0)
 			(effects
@@
 			(project ""
 				(path "/f015d259-36b1-4d36-b25a-c9dc3131b66c"
-					(reference "C_VDD_MPU1")
+					(reference "C_MPU_VDD")
 					(unit 1)
 				)
@@
 			)
 		)
-		(property "Footprint" "TCLib:C_5mm"
+		(property "Footprint" "TCLib:C_0805"
 			(at 92.71 161.798 0)
 			(effects
@@
 			)
 		)
-		(property "Description" "Unpolarized capacitor"
+		(property "Description" ""
 			(at 91.948 157.226 0)
 			(effects
