File: SRAD_computer/SRAD_computer.kicad_sch (KiCad schematic)
At the start: 49 parts, among them J1 USB_B_Micro, J2 Conn_01x02, U1 NCP1117-3.3_SOT223, U2 W25Q128JVS, U3 RP2040, U4 BME280, U5 MPU-9250, U6 SAM-M8Q-0-10, Y1 ABM8-272-T3

Commit message: RP2040 decoupling capacitors and resistances connection
Parts:
- C10, C11, C12, C13, C14, C15, C16, C2, C3, C5, C6, C7, C8, C9: footprint Capacitor_SMD:C_0402_1005Metric -> Capacitor_SMD:C_0805_2012Metric
- R3, R4, R5: footprint Resistor_SMD:R_0402_1005Metric -> Resistor_SMD:R_0805_2012Metric
Changed lines of the file:
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@@
 			)
 		)
-		(property "Footprint" "Capacitor_SMD:C_0402_1005Metric"
+		(property "Footprint" "Capacitor_SMD:C_0805_2012Metric"
 			(at 97.4852 67.31 0)
 			(effects
@@
 			)
 		)
-		(property "Footprint" "Resistor_SMD:R_0402_1005Metric"
+		(property "Footprint" "Resistor_SMD:R_0805_2012Metric"
 			(at 304.8 69.342 90)
 			(effects
@@
 			)
 		)
-		(property "Footprint" "Resistor_SMD:R_0402_1005Metric"
+		(property "Footprint" "Resistor_SMD:R_0805_2012Metric"
 			(at 304.8 76.962 90)
 			(effects
@@
 			)
 		)
-		(property "Footprint" "Capacitor_SMD:C_0402_1005Metric"
+		(property "Footprint" "Capacitor_SMD:C_0805_2012Metric"
 			(at 284.1752 44.45 0)
 			(effects
@@
 			)
 		)
-		(property "Footprint" "Capacitor_SMD:C_0402_1005Metric"
+		(property "Footprint" "Capacitor_SMD:C_0805_2012Metric"
 			(at 295.6052 44.45 0)
 			(effects
@@
 			)
 		)
-		(property "Footprint" "Capacitor_SMD:C_0402_1005Metric"
+		(property "Footprint" "Capacitor_SMD:C_0805_2012Metric"
 			(at 307.0352 44.45 0)
 			(effects
@@
 			)
 		)
-		(property "Footprint" "Capacitor_SMD:C_0402_1005Metric"
+		(property "Footprint" "Capacitor_SMD:C_0805_2012Metric"
 			(at 318.4652 44.45 0)
 			(effects
@@
 			)
 		)
-		(property "Footprint" "Capacitor_SMD:C_0402_1005Metric"
+		(property "Footprint" "Capacitor_SMD:C_0805_2012Metric"
 			(at 329.8952 44.45 0)
 			(effects
@@
 			)
 		)
-		(property "Footprint" "Capacitor_SMD:C_0402_1005Metric"
+		(property "Footprint" "Capacitor_SMD:C_0805_2012Metric"
 			(at 341.3252 44.45 0)
 			(effects
@@
 			)
 		)
-		(property "Footprint" "Capacitor_SMD:C_0402_1005Metric"
+		(property "Footprint" "Capacitor_SMD:C_0805_2012Metric"
 			(at 352.7552 44.45 0)
 			(effects
@@
 			)
 		)
-		(property "Footprint" "Capacitor_SMD:C_0402_1005Metric"
+		(property "Footprint" "Capacitor_SMD:C_0805_2012Metric"
 			(at 218.1352 44.45 0)
 			(effects
@@
 			)
 		)
-		(property "Footprint" "Capacitor_SMD:C_0402_1005Metric"
+		(property "Footprint" "Capacitor_SMD:C_0805_2012Metric"
 			(at 229.5652 44.45 0)
 			(effects
@@
 			)
 		)
-		(property "Footprint" "Capacitor_SMD:C_0402_1005Metric"
+		(property "Footprint" "Capacitor_SMD:C_0805_2012Metric"
 			(at 229.5652 59.69 0)
 			(effects
@@
 			)
 		)
-		(property "Footprint" "Capacitor_SMD:C_0402_1005Metric"
+		(property "Footprint" "Capacitor_SMD:C_0805_2012Metric"
 			(at 284.1752 59.69 0)
 			(effects
@@
 			)
 		)
-		(property "Footprint" "Capacitor_SMD:C_0402_1005Metric"
+		(property "Footprint" "Capacitor_SMD:C_0805_2012Metric"
 			(at 25.4 106.3752 0)
 			(effects
@@
 			)
 		)
-		(property "Footprint" "Resistor_SMD:R_0402_1005Metric"
+		(property "Footprint" "Resistor_SMD:R_0805_2012Metric"
 			(at 62.23 113.792 90)
 			(effects
@@
 			)
 		)
-		(property "Footprint" "Capacitor_SMD:C_0402_1005Metric"
+		(property "Footprint" "Capacitor_SMD:C_0805_2012Metric"
 			(at 25.4 116.5352 0)
 			(effects

Commit message: update PCB
Parts:
- C_BME_VDDIO1, C_MPU_REG1, C_VDDIO_MPU1, C_VDD_MPU1: footprint TCLib:C_5mm -> TCLib:C_0805
- H1, H2, H3, H4: footprint MountingHole:MountingHole_2.7mm_M2.5 -> MountingHole:MountingHole_3.5mm; now left out of the parts list
Changed lines of the file:
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@@
 		(unit 1)
 		(exclude_from_sim no)
-		(in_bom yes)
+		(in_bom no)
 		(on_board yes)
 		(dnp no)
@@
 			)
 		)
-		(property "Footprint" "MountingHole:MountingHole_2.7mm_M2.5"
+		(property "Footprint" "MountingHole:MountingHole_3.5mm"
 			(at 351.79 135.89 0)
 			(effects
@@
 		(unit 1)
 		(exclude_from_sim no)
-		(in_bom yes)
+		(in_bom no)
 		(on_board yes)
 		(dnp no)
@@
 			)
 		)
-		(property "Footprint" "MountingHole:MountingHole_2.7mm_M2.5"
+		(property "Footprint" "MountingHole:MountingHole_3.5mm"
 			(at 351.79 140.97 0)
 			(effects
@@
 		(unit 1)
 		(exclude_from_sim no)
-		(in_bom yes)
+		(in_bom no)
 		(on_board yes)
 		(dnp no)
@@
 			)
 		)
-		(property "Footprint" "MountingHole:MountingHole_2.7mm_M2.5"
+		(property "Footprint" "MountingHole:MountingHole_3.5mm"
 			(at 351.79 146.05 0)
 			(effects
@@
 		(unit 1)
 		(exclude_from_sim no)
-		(in_bom yes)
+		(in_bom no)
 		(on_board yes)
 		(dnp no)
@@
 			)
 		)
-		(property "Footprint" "MountingHole:MountingHole_2.7mm_M2.5"
+		(property "Footprint" "MountingHole:MountingHole_3.5mm"
 			(at 351.79 151.13 0)
 			(effects
@@
 			)
 		)
-		(property "Footprint" "TCLib:C_5mm"
+		(property "Footprint" "TCLib:C_0805"
 			(at 81.28 248.158 0)
 			(effects
@@
 			)
 		)
-		(property "Description" "Unpolarized capacitor"
+		(property "Description" ""
 			(at 80.518 243.586 0)
 			(effects
@@
 			)
 		)
-		(property "Footprint" "TCLib:C_5mm"
+		(property "Footprint" "TCLib:C_0805"
 			(at 93.98 237.998 0)
 			(effects
@@
 			)
 		)
-		(property "Description" "Unpolarized capacitor"
+		(property "Description" ""
 			(at 93.218 233.426 0)
 			(effects
@@
 			)
 		)
-		(property "Footprint" "TCLib:C_5mm"
+		(property "Footprint" "TCLib:C_0805"
 			(at 77.47 224.028 0)
 			(effects
@@
 			)
 		)
-		(property "Description" "Unpolarized capacitor"
+		(property "Description" ""
 			(at 76.708 219.456 0)
 			(effects
@@
 			)
 		)
-		(property "Footprint" "TCLib:C_5mm"
+		(property "Footprint" "TCLib:C_0805"
 			(at 92.71 161.798 0)
 			(effects
@@
 			)
 		)
-		(property "Description" "Unpolarized capacitor"
+		(property "Description" ""
 			(at 91.948 157.226 0)
 			(effects

Commit message: Update PCB placement & 3D models added
Parts:
- removed J1: USB_B_Micro, RP2040_minimal_r2:USB_Micro-B_Amphenol_10103594-0001LF_Horizontal_modified, symbol Connector:USB_B_Micro
- added J1: Terminal_3, TCLib:Bornera_3_P5mm, symbol TCLib:Terminal_3
- added J3: UJ20-C-H-G-SMT-1-P16-TR, my_lib:USB-C-samesky, symbol UJ20-C-H-G-SMT-1-P16-TR:UJ20-C-H-G-SMT-1-P16-TR
- added J4: Terminal_2, TCLib:Bornera_2_P5mm, symbol TCLib:Terminal_2
- added Q1: MMBT5551L, Package_TO_SOT_SMD:SOT-23, symbol Transistor_BJT:MMBT5551L
- added Q3: FDN340P, Package_TO_SOT_SMD:SOT-23, symbol Transistor_FET:FDN340P
- added R6, R7, R8: R, TCLib:R_0805, symbol Device:R
Connections:
- net BME_SCL is gone; now on net SCL: R_BME_SCL1.2, U4.4 (SCK)
- net BME_SDA is gone; now on net SDA: R_BME_SDA1.2, U4.3 (SDI)
- net +3V3: now also J1.3, Q3.2 (S), R6.1
- net GND: now also J1.2, J3.A1_B12 (GND), J3.B1_A12 (GND__1), J3.SH1 (SHIELD), J3.SH2 (SHIELD__1), J3.SH3 (SHIELD__2), J3.SH4 (SHIELD__3), J4.1, Q1.2 (E)
- net USB_D+: now also J3.A7 (DN1), J3.B7 (DN2)
- net USB_D-: now also J3.A6 (DP1), J3.B6 (DP2)
- net VBUS: now also J3.A4_B9 (VBUS), J4.2
- net SCL: now reaches R_SAM_SCL1.2, U6.12 (SCL)
- net SCL: now also R_MPU_SCL1.2, U5.23 (SCL/SCLK)
- net SDA: now reaches R_SAM_SDA1.2, U6.9 (SDA)
- net SDA: now also R_MPU_SDA1.2, U5.24 (SDA/SDI)
- new net: Q3.1 (G), R6.2, R7.1
- new net: Q1.1 (B), R8.2
- new net: Q1.3 (C), R7.2
- new net V_cam: J1.1, Q3.3 (D)
- new net power_cam: R8.1
- no-connect marks 14 -> 13
Other:
- note added: "POWER CAM"
- note removed: "Flash"
- moved on the sheet: C1, C4, C5, H1, H2, H3, H4, J2, R1, R2, U1, U2

Commit message: PCB v1
Connections:
- net SCL is gone; now on net GPIO17: R_BME_SCL1.2, R_MPU_SCL1.2, R_SAM_SCL1.2, U4.4 (SCK), U5.23 (SCL/SCLK), U6.12 (SCL)
- net SDA is gone; now on net GPIO16: R_BME_SDA1.2, R_MPU_SDA1.2, R_SAM_SDA1.2, U4.3 (SDI), U5.24 (SDA/SDI), U6.9 (SDA)
- net power_cam is gone; now on net GPIO18: R8.1
- net +3V3: no longer J1.3, Q3.2 (S), R6.1
- net GND: now also U4.5 (SDO)
- net VBUS: now also J1.3, Q3.2 (S), R6.1
Changed lines of the file:
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@@
 	(wire
 		(pts
-			(xy 289.56 132.08) (xy 304.8 132.08)
+			(xy 289.56 132.08) (xy 308.61 132.08)
 		)
 		(stroke
@@
 	(wire
 		(pts
-			(xy 289.56 127) (xy 304.8 127)
+			(xy 289.56 127) (xy 308.61 127)
 		)
 		(stroke
@@
 	(wire
 		(pts
-			(xy 289.56 129.54) (xy 304.8 129.54)
+			(xy 289.56 129.54) (xy 308.61 129.54)
 		)
 		(stroke
@@
 		)
 	)
+	(label "SDA"
+		(at 308.61 127 0)
+		(effects
+			(font
+				(size 1.27 1.27)
+			)
+			(justify left bottom)
+		)
+	)
 	(label "GPIO29_ADC3"
 		(at 304.8 162.56 180)
@@
 		)
 	)
+	(label "power_cam"
+		(at 308.61 132.08 0)
+		(effects
+			(font
+				(size 1.27 1.27)
+			)
+			(justify left bottom)
+		)
+	)
 	(label "SDA"
 		(at 148.59 254 0)
@@
 		)
 	)
+	(label "SCL"
+		(at 308.61 129.54 0)
+		(effects
+			(font
+				(size 1.27 1.27)
+			)
+			(justify left bottom)
+		)
+	)
 	(label "USB_D-"
 		(at 322.58 78.74 180)
@@
 	)
 	(symbol
+		(lib_id "power:VBUS")
+		(at 354.33 93.98 0)
+		(unit 1)
+		(exclude_from_sim no)
+		(in_bom yes)
+		(on_board yes)
+		(dnp no)
+		(property "Reference" "#PWR045"
+			(at 354.33 97.79 0)
+			(effects
+				(font
+					(size 1.27 1.27)
+				)
+				(hide yes)
+			)
+		)
+		(property "Value" "VBUS"
+			(at 354.711 89.5858 0)
+			(effects
+				(font
+					(size 1.27 1.27)
+				)
+			)
+		)
+		(property "Footprint" ""
+			(at 354.33 93.98 0)
+			(effects
+				(font
+					(size 1.27 1.27)
+				)
+				(hide yes)
+			)
+		)
+		(property "Datasheet" ""
+			(at 354.33 93.98 0)
+			(effects
+				(font
+					(size 1.27 1.27)
+				)
+				(hide yes)
+			)
+		)
+		(property "Description" ""
+			(at 354.33 93.98 0)
+			(effects
+				(font
+					(size 1.27 1.27)
+				)
+			)
+		)
+		(pin "1"
+		)
+		(instances
+			(project "SRAD_computer"
+				(path "/f015d259-36b1-4d36-b25a-c9dc3131b66c"
+					(reference "#PWR045")
+					(unit 1)
+				)
+			)
+		)
+	)
+	(symbol
 		(lib_id "power:+3V3")
 		(at 110.49 236.22 0)
@@
 	)
 	(symbol
-		(lib_id "power:+3V3")
-		(at 354.33 93.98 0)
-		(unit 1)
-		(exclude_from_sim no)
-		(in_bom yes)
-		(on_board yes)
-		(dnp no)
-		(property "Reference" "#PWR040"
-			(at 354.33 97.79 0)
-			(effects
-				(font
-					(size 1.27 1.27)
-				)
-				(hide yes)
-			)
-		)
-		(property "Value" "+3V3"
-			(at 354.711 89.5858 0)
-			(effects
-				(font
-					(size 1.27 1.27)
-				)
-			)
-		)
-		(property "Footprint" ""
-			(at 354.33 93.98 0)
-			(effects
-				(font
-					(size 1.27 1.27)
-				)
-				(hide yes)
-			)
-		)
-		(property "Datasheet" ""
-			(at 354.33 93.98 0)
-			(effects
-				(font
-					(size 1.27 1.27)
-				)
-				(hide yes)
-			)
-		)
-		(property "Description" ""
-			(at 354.33 93.98 0)
-			(effects
-				(font
-					(size 1.27 1.27)
-				)
-			)
-		)
-		(pin "1"
-		)
-		(instances
-			(project "SRAD_computer"
-				(path "/f015d259-36b1-4d36-b25a-c9dc3131b66c"
-					(reference "#PWR040")
-					(unit 1)
-				)
-			)
-		)
-	)
-	(symbol
 		(lib_id "TCLib:C")
 		(at 97.79 165.1 0)
@@
 					(unit 1)
 				)
+			)
+		)
+	)
+	(symbol
+		(lib_name "GND_15")
+		(lib_id "power:GND")
+		(at 64.77 173.99 0)
+		(unit 1)
+		(exclude_from_sim no)
+		(in_bom yes)
+		(on_board yes)
+		(dnp no)
+		(fields_autoplaced yes)
+		(property "Reference" "#PWR044"
+			(at 64.77 180.34 0)
+			(effects
+				(font
+					(size 1.27 1.27)
+				)
+				(hide yes)
+			)
+		)
+		(property "Value" "GND"
+			(at 64.77 179.07 0)
+			(effects
+				(font
+					(size 1.27 1.27)
+				)
+			)
+		)
+		(property "Footprint" ""
+			(at 64.77 173.99 0)
+			(effects
+				(font
+					(size 1.27 1.27)
+				)
+				(hide yes)
+			)
+		)
+		(property "Datasheet" ""
+			(at 64.77 173.99 0)
+			(effects
+				(font
+					(size 1.27 1.27)
+				)
+				(hide yes)
+			)
+		)
+		(property "Description" "Power symbol creates a global label with name \"GND\" , ground"
+			(at 64.77 173.99 0)
+			(effects
+				(font
+					(size 1.27 1.27)
+				)
+				(hide yes)
+			)
+		)
+		(pin "1"
+		)
+		(instances
+			(project ""
+				(path "/f015d259-36b1-4d36-b25a-c9dc3131b66c"
+					(reference "#PWR044")
+					(unit 1)
+				)

Commit message: SD slot, LEDs and switch added
Parts:
- removed Y1: ABM8-272-T3, Crystal:Crystal_SMD_3225-4Pin_3.2x2.5mm, symbol Device:Crystal_GND24
- added D1, D2, D3: LED, LED_SMD:LED_0805_2012Metric_Pad1.15x1.40mm_HandSolder, symbol Device:LED
- added J5: Connector_3_Pol, TCLib:Molex_1x03_P2.54mm, symbol TCLib:Connector_3_Pol
- added J6: Micro_SD_Card, Connector_Card:microSD_HC_Wuerth_693072010801, symbol Connector:Micro_SD_Card
- added R10, R11, R12: R, TCLib:R_0805, symbol Device:R
- added R9: R, Resistor_SMD:R_0805_2012Metric_Pad1.20x1.40mm_HandSolder, symbol Device:R
- added S1: PTS810SJK250SMTR_LFS, PTS810SJK250SMTRLFS, symbol Rocketry_FC:PTS810SJK250SMTR_LFS
- added Y1: Crystal, Crystal:Crystal_HC49-4H_Vertical, symbol Device:Crystal
Connections:
- net GND: now also J5.3, J6.9 (SHIELD), R10.2, R11.2, R12.2, R9.2
- net VBUS: no longer J1.3, Q3.2 (S), R6.1
- net XIN: now also Y1.2
- net at C3.1, R5.2: now also Y1.1
- net GPIO10 renamed LED_2
- net LED_2: now also D2.2 (A)
- net GPIO11 renamed LED_1
- net LED_1: now also D1.2 (A)
- net GPIO16 renamed SDA
- net GPIO17 renamed SCL
- net GPIO18 renamed power_cam
- net GPIO19 renamed UART_Tx
- net UART_Tx: now also J5.2
- net GPIO20 renamed UART_Rx
- net UART_Rx: now also J5.1
- net GPIO23 renamed SW_1
- net SW_1: now also S1.1 (NO_1), S1.2 (NO_2)
- net GPIO9 renamed LED_3
- net LED_3: now also D3.2 (A)
- new net: D1.1 (K), R9.1
- new net: R12.1, S1.3 (COM_1), S1.4 (COM_2)
- new net: D3.1 (K), R11.1
- new net: D2.1 (K), R10.1
- new net V_cam_bus: J1.3, Q3.2 (S), R6.1
Other:
- moved on the sheet: H1, H2, H3, H4

Commit message: PCB 3D model added
Parts:
- J6: footprint Connector_Card:microSD_HC_Wuerth_693072010801 -> my_lib:microSD_HC_Wuerth_693072010801
Changed lines of the file:
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@@
 			)
 		)
-		(property "Footprint" "Connector_Card:microSD_HC_Wuerth_693072010801"
+		(property "Footprint" "my_lib:microSD_HC_Wuerth_693072010801"
 			(at 334.01 196.85 0)
 			(effects

Commit message: PCB V2 first draft
Parts:
- J6: footprint my_lib:microSD_HC_Wuerth_693072010801 -> my_lib:microSD_HC_Molex_47219-2001
Connections:
- net GPIO21 is gone; now on net SD_CLK: U3.32 (GPIO21)
- net GPIO22 is gone; now on net SD_CMD: U3.34 (GPIO22)
- net GPIO25 is gone; now on net SD_DAT2: U3.37 (GPIO25)
- net GPIO26_ADC0 is gone; now on net UART_Tx: U3.38 (GPIO26_ADC0)
- net GPIO27_ADC1 is gone; now on net UART_Rx: U3.39 (GPIO27_ADC1)
- net GPIO28_ADC2 is gone; now on net SW_1: U3.40 (GPIO28_ADC2)
- net GPIO29_ADC3 is gone; now on net power_cam: U3.41 (GPIO29_ADC3)
- net SW_1: no longer U3.35 (GPIO23)
- net UART_Rx: no longer U3.31 (GPIO20)
- net UART_Tx: no longer U3.30 (GPIO19)
- net power_cam: no longer U3.29 (GPIO18)
- net SD_DAT2: now reaches J6.1 (DAT2)
- net SD_DAT3: now reaches J6.2 (DAT3/CD)
- net SD_DAT3: now also U3.35 (GPIO23)
- net SD_CMD: now reaches J6.3 (CMD)
- net SD_CLK: now reaches J6.5 (CLK)
- net SD_VSS: now reaches J6.6 (VSS)
- net SD_VSS: now also U3.31 (GPIO20)
- net SD_DAT0: now reaches J6.7 (DAT0)
- net SD_DAT0: now also U3.30 (GPIO19)
- net SD_DAT1: now reaches J6.8 (DAT1)
- net SD_DAT1: now also U3.29 (GPIO18)
Changed lines of the file:
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@@
 	(wire
 		(pts
+			(xy 269.24 196.85) (xy 281.94 196.85)
+		)
+		(stroke
+			(width 0)
+			(type default)
+		)
+	)
+	(wire
+		(pts
 			(xy 21.59 236.22) (xy 29.21 236.22)
 		)
@@
 	(wire
 		(pts
+			(xy 269.24 212.09) (xy 281.94 212.09)
+		)
+		(stroke
+			(width 0)
+			(type default)
+		)
+	)
+	(wire
+		(pts
 			(xy 289.56 104.14) (xy 304.8 104.14)
 		)
@@
 	(wire
 		(pts
+			(xy 269.24 214.63) (xy 281.94 214.63)
+		)
+		(stroke
+			(width 0)
+			(type default)
+		)
+	)
+	(wire
+		(pts
 			(xy 146.05 233.68) (xy 146.05 236.22)
 		)
@@
 	(wire
 		(pts
+			(xy 269.24 209.55) (xy 281.94 209.55)
+		)
+		(stroke
+			(width 0)
+			(type default)
+		)
+	)
+	(wire
+		(pts
 			(xy 283.21 44.45) (xy 283.21 46.99)
 		)
@@
 	(wire
 		(pts
+			(xy 269.24 199.39) (xy 281.94 199.39)
+		)
+		(stroke
+			(width 0)
+			(type default)
+		)
+	)
+	(wire
+		(pts
 			(xy 85.09 27.94) (xy 95.25 27.94)
 		)
@@
 	(wire
 		(pts
+			(xy 269.24 207.01) (xy 281.94 207.01)
+		)
+		(stroke
+			(width 0)
+			(type default)
+		)
+	)
+	(wire
+		(pts
 			(xy 121.92 63.5) (xy 138.43 63.5)
 		)
@@
 	(wire
 		(pts
+			(xy 269.24 201.93) (xy 281.94 201.93)
+		)
+		(stroke
+			(width 0)
+			(type default)
+		)
+	)
+	(wire
+		(pts
 			(xy 328.93 154.94) (xy 337.82 154.94)
 		)
@@
 		)
 	)
-	(label "GPIO27_ADC1"
+	(label "UART_Rx"
 		(at 304.8 157.48 180)
 		(effects
@@
 		)
 	)
-	(label "SW_1"
+	(label "SD_DAT3"
 		(at 304.8 144.78 180)
 		(effects
@@
 		)
 	)
+	(label "SD_CLK"
+		(at 269.24 207.01 0)
+		(effects
+			(font
+				(size 1.27 1.27)
+			)
+			(justify left bottom)
+		)
+	)
 	(label "USB_D+"
 		(at 52.07 35.56 180)
@@
 		)
 	)
-	(label "GPIO29_ADC3"
+	(label "power_cam"
 		(at 304.8 162.56 180)
 		(effects
@@
 		)
 	)
-	(label "GPIO22"
+	(label "SD_CMD"
 		(at 304.8 142.24 180)
 		(effects
@@
 		)
 	)
-	(label "GPIO26_ADC0"
+	(label "UART_Tx"
 		(at 304.8 154.94 180)
 		(effects
@@
 		)
 	)
+	(label "SD_DAT1"
+		(at 269.24 214.63 0)
+		(effects
+			(font
+				(size 1.27 1.27)
+			)
+			(justify left bottom)
+		)
+	)
 	(label "USB_D-"
 		(at 52.07 38.1 180)
@@
 		)
 	)
-	(label "power_cam"
+	(label "SD_DAT1"
 		(at 304.8 132.08 180)
 		(effects
@@
 		)
 	)
+	(label "SD_DAT3"
+		(at 269.24 199.39 0)
+		(effects
+			(font
+				(size 1.27 1.27)
+			)
+			(justify left bottom)
+		)
+	)
 	(label "QSPI_SD2"
 		(at 121.92 71.12 0)
@@
 		)
 	)
+	(label "SD_VSS"
+		(at 269.24 209.55 0)
+		(effects
+			(font
+				(size 1.27 1.27)
+			)
+			(justify left bottom)
+		)
+	)
 	(label "USB_D+"
 		(at 322.58 71.12 180)
@@
 		)
 	)
+	(label "SD_DAT0"
+		(at 269.24 212.09 0)
+		(effects
+			(font
+				(size 1.27 1.27)
+			)
+			(justify left bottom)
+		)
+	)
 	(label "QSPI_SD3"
 		(at 212.09 99.06 0)
@@
 		)
 	)
-	(label "UART_Rx"
+	(label "SD_VSS"
 		(at 304.8 137.16 180)
 		(effects
@@
 		)
 	)
-	(label "GPIO28_ADC2"
+	(label "SW_1"
 		(at 304.8 160.02 180)
 		(effects
@@
 		)
 	)
-	(label "GPIO21"
+	(label "SD_CMD"
+		(at 269.24 201.93 0)
+		(effects
+			(font
+				(size 1.27 1.27)
+			)
+			(justify left bottom)
+		)
+	)
+	(label "SD_CLK"
 		(at 304.8 139.7 180)
 		(effects
@@
 		)
 	)
-	(label "GPIO25"
+	(label "SD_DAT2"
+		(at 269.24 196.85 0)
+		(effects
+			(font
+				(size 1.27 1.27)
+			)
+			(justify left bottom)
+		)
+	)
+	(label "SD_DAT2"
 		(at 304.8 149.86 180)
 		(effects
@@
 		)
 	)
-	(label "UART_Tx"
+	(label "SD_DAT0"
 		(at 304.8 134.62 180)
 		(effects
@@
 			)
 		)
-		(property "Footprint" "my_lib:microSD_HC_Wuerth_693072010801"
+		(property "Footprint" "my_lib:microSD_HC_Molex_47219-2001"
 			(at 334.01 196.85 0)
 			(effects

Commit message: changes in USB pins. D+ -> D-
Connections:
- net USB_D+: now also J3.A6 (DP1), J3.B6 (DP2); no longer J3.A7 (DN1), J3.B7 (DN2)
- net USB_D-: now also J3.A7 (DN1), J3.B7 (DN2); no longer J3.A6 (DP1), J3.B6 (DP2)
Changed lines of the file:
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@@
 		)
 	)
-	(label "USB_D+"
+	(label "USB_D-"
 		(at 52.07 35.56 180)
 		(effects
@@
 		)
 	)
-	(label "USB_D-"
+	(label "USB_D+"
 		(at 52.07 38.1 180)
 		(effects
@@
 		)
 	)
-	(label "USB_D-"
+	(label "USB_D+"
 		(at 52.07 45.72 180)
 		(effects
@@
 		)
 	)
-	(label "USB_D+"
+	(label "USB_D-"
 		(at 52.07 43.18 180)
 		(effects
