File: SRAD_computer/SRAD_computer.kicad_pcb (KiCad board)
At the start: 2 copper layers, 90 x 80 mm, 71 parts, among them J1 Terminal_3, J2 Conn_01x02, J3 UJ20-C-H-G-SMT-1-P16-TR, J4 Terminal_2, J5 Connector_3_Pol, J6 Micro_SD_Card, Q1 MMBT5551L, Q3 FDN340P, U1 NCP1117-3.3_SOT223, U2 W25Q128JVS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

Commit message: .
Parts:
- moved H3 75.8 mm to (128.4, 117.8), turned to 0 degrees
- moved H2 73.1 mm to (128.4, 42.8), turned to 0 degrees
- moved H4 67.7 mm to (63.4, 117.8), turned to 0 degrees
- moved J4 66.6 mm to (118.8, 40.6), turned to 180 degrees
- moved H1 64.7 mm to (63.4, 42.8), turned to 0 degrees
- moved G*** 63.0 mm to (128.2, 104.2), turned to 90 degrees
- moved C4 62.7 mm to (127.9, 53.8), turned to -90 degrees
- moved J5 61.3 mm to (131.8, 63.1), turned to -90 degrees
- moved J3 61.0 mm to (101.4, 37.1), turned to 180 degrees
- moved J2 59.3 mm to (69.8, 43.0), turned to 180 degrees
- moved R15 59.0 mm to (133.1, 76.5), turned to -90 degrees
- moved U1 57.1 mm to (120.4, 50.8), turned to 0 degrees
- moved C18 55.2 mm to (130.4, 76.6), turned to -90 degrees
- moved J1 55.0 mm to (87.5, 40.3), turned to 180 degrees
- moved C17 54.6 mm to (94.6, 40.5), turned to -90 degrees
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Other:
- board size 90 x 80 mm -> 80 x 90 mm
