File: SRAD_Design/SRAD_computer.kicad_pcb (KiCad board)
At the start: 2 copper layers, 80 x 90 mm, 71 parts, among them J1 Connector_2_Pol, J2 503398-1892, J4 Terminal_2, J5 Connector_3_Pol, J7 UJ20-C-H-G-SMT-6-P16-TR, U1 NCP1117-3.3_SOT223, U2 W25Q128JVS, U3 RP2040, U4 BME280, U5 MPU-9250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

Commit message: IMU fixed
Connections:
- J5 pad 1: /UART_Rx -> /UART_Tx
- J5 pad 2: /UART_Tx -> /UART_Rx
- U3 pad 36: /SD_DAT1 -> /UART_Tx
- U3 pad 37: /UART_Tx -> /UART_Rx
- U3 pad 38: /UART_Rx -> /SD_DAT1
Routing:
- net /UART_Rx: track 50.5 -> 100.1 mm, vias 1 -> 2
- net /SD_DAT1: track 83.3 -> 36.6 mm
- net /UART_Tx: track 49.6 -> 43.8 mm, vias 1 -> 0

Commit message: Updated PCB: some UART pin errors & missing conection on icm
Parts:
- moved R12 1.85 mm to (123.6, 66.3)
Connections:
- J5 pad 1: /UART_Tx -> /UART_Rx
- J5 pad 2: /UART_Rx -> /UART_Tx
- U5 pad 9: unconnected-(U5-AD0/SDO-Pad9) -> +3V3
Routing:
- net /SD_DAT1: track 36.6 -> 98.2 mm
- net /UART_Rx: track 100.1 -> 50.8 mm, vias 2 -> 0
- net /UART_Tx: track 43.8 -> 49.8 mm
- net +3V3: track 621.0 -> 623.6 mm
Other:
- board text added: "GND"
- board text added: "ITBA Rocketry team - A&R Hertter, Jose Ivan Diaz Guzmán, Ezequiel 2025"
- board text added: "Rx"
- board text added: "Tx"
- board text removed: "ITBA Rocketry team - A&R Hertter, Jose Ivan Diaz Guzmán, Ezequiel"

Commit message: Airbrake function
Connections:
- net /servo renamed /AIRBRAKE
