File: SRAD_Design/SRAD_computer.kicad_sch (KiCad schematic)
At the start: 69 parts, among them J1 Connector_2_Pol, J2 503398-1892, J4 Terminal_2, J5 Connector_3_Pol, J7 UJ20-C-H-G-SMT-6-P16-TR, U1 NCP1117-3.3_SOT223, U2 W25Q128JVS, U3 RP2040, U4 BME280, U5 MPU-9250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

Commit message: IMU fixed
Connections:
- net +3V3: now also U5.9 (AD0/SDO)
- net SD_DAT1: now also U3.38 (GPIO26_ADC0); no longer U3.36 (GPIO24)
- net UART_Rx: now also J5.2, U3.37 (GPIO25); no longer J5.1, U3.38 (GPIO26_ADC0)
- net UART_Tx: now also J5.1, U3.36 (GPIO24); no longer J5.2, U3.37 (GPIO25)
Changed lines of the file:
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@@
 	(wire
 		(pts
+			(xy 34.29 255.27) (xy 41.91 255.27)
+		)
+		(stroke
+			(width 0)
+			(type default)
+		)
+	)
+	(wire
+		(pts
 			(xy 69.85 59.69) (xy 100.33 59.69)
 		)
@@
 	(wire
 		(pts
+			(xy 34.29 255.27) (xy 34.29 260.35)
+		)
+		(stroke
+			(width 0)
+			(type default)
+		)
+	)
+	(wire
+		(pts
 			(xy 261.62 143.51) (xy 247.65 143.51)
 		)
@@
 	(wire
 		(pts
+			(xy 34.29 260.35) (xy 27.94 260.35)
+		)
+		(stroke
+			(width 0)
+			(type default)
+		)
+	)
+	(wire
+		(pts
 			(xy 261.62 77.47) (xy 247.65 77.47)
 		)
@@
 		)
 	)
-	(label "SD_DAT1"
+	(label "UART_Tx"
 		(at 340.36 137.16 180)
 		(effects
@@
 		)
 	)
-	(label "UART_Rx"
+	(label "SD_DAT1"
 		(at 340.36 144.78 180)
 		(effects
@@
 		)
 	)
-	(label "UART_Rx"
+	(label "UART_Tx"
 		(at 298.45 195.58 0)
 		(effects
@@
 		)
 	)
-	(label "UART_Tx"
+	(label "UART_Rx"
 		(at 340.36 139.7 180)
 		(effects
@@
 		)
 	)
-	(label "UART_Tx"
+	(label "UART_Rx"
 		(at 298.45 193.04 0)
 		(effects
@@
 					(unit 1)
 				)
+			)
+		)
+	)
+	(symbol
+		(lib_id "power:+3V3")
+		(at 27.94 260.35 0)
+		(unit 1)
+		(exclude_from_sim no)
+		(in_bom yes)
+		(on_board yes)
+		(dnp no)
+		(property "Reference" "#PWR041"
+			(at 27.94 264.16 0)
+			(effects
+				(font
+					(size 1.27 1.27)
+				)
+				(hide yes)
+			)
+		)
+		(property "Value" "+3V3"
+			(at 28.321 255.9558 0)
+			(effects
+				(font
+					(size 1.27 1.27)
+				)
+			)
+		)
+		(property "Footprint" ""
+			(at 27.94 260.35 0)
+			(effects
+				(font
+					(size 1.27 1.27)
+				)
+				(hide yes)
+			)
+		)
+		(property "Datasheet" ""
+			(at 27.94 260.35 0)
+			(effects
+				(font
+					(size 1.27 1.27)
+				)
+				(hide yes)
+			)
+		)
+		(property "Description" ""
+			(at 27.94 260.35 0)
+			(effects
+				(font
+					(size 1.27 1.27)
+				)
+			)
+		)
+		(pin "1"
+		)
+		(instances
+			(project "SRAD_computer"
+				(path "/f015d259-36b1-4d36-b25a-c9dc3131b66c"
+					(reference "#PWR041")
+					(unit 1)
+				)

Commit message: Updated PCB: some UART pin errors & missing conection on icm
Parts:
- J2: footprint my_lib:503398-1892-1 -> my_lib:693071010811
Connections:
- net UART_Rx: now also J5.1; no longer J5.2
- net UART_Tx: now also J5.2; no longer J5.1
Changed lines of the file:
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@@
 		)
 	)
-	(label "UART_Tx"
+	(label "UART_Rx"
 		(at 298.45 195.58 0)
 		(effects
@@
 		)
 	)
-	(label "UART_Rx"
+	(label "UART_Tx"
 		(at 298.45 193.04 0)
 		(effects
@@
 			)
 		)
-		(property "Footprint" "my_lib:503398-1892-1"
+		(property "Footprint" "my_lib:693071010811"
 			(at 201.93 260.02 0)
 			(effects

Commit message: Airbrake function
Connections:
- net servo renamed AIRBRAKE
Changed lines of the file:
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@@
 		)
 	)
-	(label "servo"
+	(label "AIRBRAKE"
 		(at 339.09 176.53 0)
 		(effects
@@
 		)
 	)
-	(label "servo"
+	(label "AIRBRAKE"
 		(at 340.36 152.4 180)
 		(effects

Commit message: fsm tested
Parts:
- R10, R11, R9: value R -> 150
- R_BL1: value R -> 15k
- R_BL2: value R -> 8k2
- R_BME_SCL1, R_BME_SDA1, R_MPU_SCL1, R_MPU_SDA1, R_SAM_SCL1, R_SAM_SDA1: value R -> 2k7
Changed lines of the file:
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@@
 			)
 		)
-		(property "Value" "R"
+		(property "Value" "15k"
 			(at 351.79 146.0499 0)
 			(effects
@@
 			)
 		)
-		(property "Value" "R"
+		(property "Value" "2k7"
 			(at 54.61 163.8299 0)
 			(effects
@@
 			)
 		)
-		(property "Value" "R"
+		(property "Value" "2k7"
 			(at 142.748 248.412 0)
 			(effects
@@
 			)
 		)
-		(property "Value" "R"
+		(property "Value" "2k7"
 			(at 157.48 246.3799 0)
 			(effects
@@
 			)
 		)
-		(property "Value" "R"
+		(property "Value" "150"
 			(at 262.89 218.4399 0)
 			(effects
@@
 			)
 		)
-		(property "Value" "R"
+		(property "Value" "150"
 			(at 285.75 218.4399 0)
 			(effects
@@
 			)
 		)
-		(property "Value" "R"
+		(property "Value" "2k7"
 			(at 38.1 163.8299 0)
 			(effects
@@
 			)
 		)
-		(property "Value" "R"
+		(property "Value" "2k7"
 			(at 24.13 247.6499 0)
 			(effects
@@
 			)
 		)
-		(property "Value" "R"
+		(property "Value" "150"
 			(at 274.32 218.4399 0)
 			(effects
@@
 			)
 		)
-		(property "Value" "R"
+		(property "Value" "8k2"
 			(at 351.79 156.2099 0)
 			(effects
@@
 			)
 		)
-		(property "Value" "R"
+		(property "Value" "2k7"
 			(at 31.75 246.3799 0)
 			(effects
